File: PsxControllerShield.kicad_pcb (KiCad board)
At the start: 2 copper layers, 68.6 x 53.3 mm, 27 parts, among them J1 TO_PSX_PAD, J2 OSHW_LOGO, Q1 BSS138, Q2 BSS138, Q3 BSS138, Q4 BSS138, Q5 BSS138, U1 LM1117-3.3

Commit message: Work in progress
Parts:
- moved Q1 1.52 mm to (151.4, 111.2)
- moved R1 1.52 mm to (157.4, 111.2)
- moved R6 1.52 mm to (145.3, 111.2)
- moved LD1 1.40 mm to (148.3, 75.6)
- moved R11 1.40 mm to (154.6, 75.6)
- moved Q2 1.02 mm to (151.4, 105.6)
- moved R2 1.02 mm to (157.4, 105.6)
- moved R7 1.02 mm to (145.3, 105.6)
- moved LD3 0.76 mm to (148.3, 81.5)
- moved R13 0.76 mm to (154.6, 81.5)
- moved R5 0.56 mm to (157.4, 89.0)
- moved Q3 0.51 mm to (151.4, 100.1)
- moved Q5 0.51 mm to (151.4, 88.9)
- moved R10 0.51 mm to (145.3, 88.9)
- moved R3 0.51 mm to (157.4, 100.1)
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Routing:
- net /ps_clk: track 26.4 -> 29.1 mm
- net /led1: track 4.57 -> 7.19 mm
- net +3V3: track 97.5 -> 96.0 mm
- net /ps_cmd: track 41.6 -> 40.6 mm
- net /led3: track 18.8 -> 18.0 mm
- net /ps_data_3v3: track 13.9 -> 13.2 mm
- net /ps_data: track 52.6 -> 52.0 mm
- net /ps_attn: track 37.8 -> 37.1 mm
- net /ps_ack_3v3: track 20.0 -> 20.5 mm
- net /ps_ack: track 24.5 -> 25.0 mm
- net /ps_attn_3v3: track 21.8 -> 21.3 mm
Other:
- board text added: "3.3V"
- board text added: "5V"
- board text added: "A0"
- board text added: "A1"
- board text added: "A2"
- board text added: "A3"
- board text added: "A4"
- board text added: "A5"
- board text added: "IOREF"
- board text added: "RESET"
- board text added: "VIN"

Commit message: Ready for protoypes!
Parts:
- moved J2 1.65 mm to (167.9, 99.4)
- moved Q3 0.58 mm to (151.4, 99.5)
- moved R3 0.58 mm to (157.4, 99.5)
- moved R8 0.58 mm to (145.3, 99.5)
- moved Q1 0.58 mm to (151.4, 110.6)
- moved Q2 0.58 mm to (151.4, 105.1)
- moved Q4 0.58 mm to (151.4, 93.9)
- moved Q5 0.58 mm to (151.4, 88.3)
- moved R1 0.58 mm to (157.4, 110.6)
- moved R10 0.58 mm to (145.3, 88.3)
- moved R2 0.58 mm to (157.4, 105.1)
- moved R4 0.58 mm to (157.4, 93.9)
- moved R5 0.58 mm to (157.4, 88.4)
- moved R6 0.58 mm to (145.3, 110.6)
- moved R7 0.58 mm to (145.3, 105.1)
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Routing:
- net /ps_cmd: track 40.6 -> 39.3 mm
- net /ps_attn_3v3: track 21.3 -> 20.6 mm
- net /ps_clk_3v3: track 18.9 -> 18.3 mm
- net /ps_ack: track 25.0 -> 24.5 mm
- net /ps_ack_3v3: track 20.5 -> 20.0 mm
Other:
- board text added: "This shield drives the PSX controller through the SPI bus. It also uses pin 9 for the ACK signal and pin 10 for ATTN. Leds are on pins 6/7/8. It also powers the vibration motors from the VIN pin. Thus it is recommended to power the Arduino board with exactly 9V through the barrel jack."
- board text added: "V1"
- board text added: "github.com/SukkoPera/PsxControllerShield Licensed under CERN OHL v.1.2"
